Commit message: Initial commit

File: p2os_urdf/defs/pioneer3dx.urdf.xacro (robot description, xacro)
@@ -5,6 +5,6 @@
 	xmlns:interface="http://playerstage.sourceforge.net/gazebo/xmlschema/#interface"
 	xmlns:xacro="http://ros.org/wiki/xacro">
-  <!--<include filename="$(find p2os_urdf)/defs/materials.xacro"/>-->
-  <include filename="$(find p2os_urdf)/defs/pioneer3dx_wheel.xacro"/>
+  <!--<xacro:include filename="$(find p2os_urdf)/defs/materials.xacro"/>-->
+  <xacro:include filename="$(find p2os_urdf)/defs/pioneer3dx_wheel.xacro"/>
 <!-- Chassis -->
 	<link name="base_link">

File: p2os_urdf/defs/pioneer3dx_body.xacro (robot description, xacro)
@@ -6,5 +6,5 @@
 	   xmlns:xacro="http://ros.org/wiki/xacro"
 	   >
-	<include filename="$(find p2os_urdf)/defs/pioneer3dx_wheel.xacro"/>
+	<xacro:include filename="$(find p2os_urdf)/defs/pioneer3dx_wheel.xacro"/>
 	<!-- Chassis description -->
 	<link name="base_link">

File: p2os_urdf/defs/pioneer3dx_wheel.xacro (robot description, xacro)
@@ -6,7 +6,7 @@
   xmlns:xacro="http://ros.org/wiki/xacro"
   >
-  <!--<include filename="$(find p2os_urdf)/defs/materials.xacro"/>-->
+  <!--<xacro:include filename="$(find p2os_urdf)/defs/materials.xacro"/>-->
   <!-- Properties (Constants) -->
-  <property name="M_PI" value="3.14159"/>
+  <xacro:property name="M_PI" value="3.14159"/>
 <!-- Right/Left Hubcap + Wheel -->
 <xacro:macro name="p3dx_wheel" params="suffix parent reflect">
